File: hw/control/cpu.sch (KiCad schematic (older format))
At the start: 33 parts, among them J301 Conn_02x05_Odd_Even, J302 Conn_01x04, J303 Raspberry_Pi_0_2_3, J304 Micro_SD_Card, J305 Conn_01x06, J306 Conn_01x07, Q301 SI2312CDS-T1-GE3, SW301 SW_Push, U301 CAT24C256

Commit message: [hw] Re-annotate all components
Parts:
- renumbered C305 to C303, C306 to C304, C304 to C305, C303 to C306, J306 to J304, J304 to J305, J305 to J306, JP304 to JP301, JP301 to JP302, JP302 to JP303, JP303 to JP304, R307 to R303, R310 to R304, R311 to R305, R312 to R306, R308 to R307, R309 to R308, R303 to R309, R304 to R310, R305 to R311, R306 to R312
