File: hw/control/led_driver.sch (KiCad schematic (older format))
At the start: 11 parts, among them U1101 SN74AHCT125D

Commit message: [hw] Re-annotate all components
Parts:
- renumbered C1101 to C1301, C1102 to C1302, R1101 to R1301, R1102 to R1302, R1103 to R1303, R1104 to R1304, R1105 to R1305, R1106 to R1306, R1107 to R1307, R1108 to R1308, U1101 to U1301
Changed lines of the file:
@@
 DATA_OUT1
 $Comp
-L SN74AHCT125D:SN74AHCT125D U1101
+L SN74AHCT125D:SN74AHCT125D U1301
 U 1 1 6146F060
 P 6300 3950
-F 0 "U1101" H 6300 4820 50  0000 C CNN
+F 0 "U1301" H 6300 4820 50  0000 C CNN
 F 1 "SN74AHCT125D" H 6300 4729 50  0000 C CNN
 F 2 "Package_SO:SO-14_3.9x8.65mm_P1.27mm" H 6300 3950 50  0001 L BNN
@@
 	5450 4350 5600 4350
 $Comp
-L power:+5V #PWR01101
+L power:+5V #PWR01301
 U 1 1 61473D10
 P 5350 2350
-F 0 "#PWR01101" H 5350 2200 50  0001 C CNN
+F 0 "#PWR01301" H 5350 2200 50  0001 C CNN
 F 1 "+5V" H 5365 2523 50  0000 C CNN
 F 2 "" H 5350 2350 50  0001 C CNN
@@
 	5350 3450 5600 3450
 $Comp
-L Device:C C1102
+L Device:C C1302
 U 1 1 6147522C
 P 4900 2700
-F 0 "C1102" H 5015 2746 50  0000 L CNN
+F 0 "C1302" H 5015 2746 50  0000 L CNN
 F 1 "10u" H 5015 2655 50  0000 L CNN
 F 2 "Capacitor_SMD:C_1206_3216Metric_Pad1.33x1.80mm_HandSolder" H 4938 2550 50  0001 C CNN
@@
 $EndComp
 $Comp
-L Device:C C1101
+L Device:C C1301
 U 1 1 61475C06
 P 4300 2700
-F 0 "C1101" H 4415 2746 50  0000 L CNN
+F 0 "C1301" H 4415 2746 50  0000 L CNN
 F 1 "100n" H 4415 2655 50  0000 L CNN
 F 2 "Capacitor_SMD:C_0805_2012Metric_Pad1.18x1.45mm_HandSolder" H 4338 2550 50  0001 C CNN
@@
 	4900 2450 5350 2450
 $Comp
-L power:GND #PWR01102
+L power:GND #PWR01302
 U 1 1 61476844
 P 4300 3100
-F 0 "#PWR01102" H 4300 2850 50  0001 C CNN
+F 0 "#PWR01302" H 4300 2850 50  0001 C CNN
 F 1 "GND" H 4305 2927 50  0000 C CNN
 F 2 "" H 4300 3100 50  0001 C CNN
@@
 	4300 2950 4300 2850
 $Comp
-L Device:R R1108
+L Device:R R1308
 U 1 1 6147BD41
 P 5150 4700
-F 0 "R1108" H 5220 4746 50  0000 L CNN
+F 0 "R1308" H 5220 4746 50  0000 L CNN
 F 1 "10K" H 5220 4655 50  0000 L CNN
 F 2 "Resistor_SMD:R_0805_2012Metric_Pad1.20x1.40mm_HandSolder" V 5080 4700 50  0001 C CNN
@@
 $EndComp
 $Comp
-L Device:R R1107
+L Device:R R1307
 U 1 1 6147C52A
 P 4750 4700
-F 0 "R1107" H 4820 4746 50  0000 L CNN
+F 0 "R1307" H 4820 4746 50  0000 L CNN
 F 1 "10K" H 4820 4655 50  0000 L CNN
 F 2 "Resistor_SMD:R_0805_2012Metric_Pad1.20x1.40mm_HandSolder" V 4680 4700 50  0001 C CNN
@@
 	4750 4550 4750 4150
 $Comp
-L power:GND #PWR01103
+L power:GND #PWR01303
 U 1 1 6147D2D2
 P 4750 5100
-F 0 "#PWR01103" H 4750 4850 50  0001 C CNN
+F 0 "#PWR01303" H 4750 4850 50  0001 C CNN
 F 1 "GND" H 4755 4927 50  0000 C CNN
 F 2 "" H 4750 5100 50  0001 C CNN
@@
 	5450 3950 5450 3850
 $Comp
-L Device:R R1103
+L Device:R R1303
 U 1 1 614BACD3
 P 3200 4150
-F 0 "R1103" V 3407 4150 50  0000 C CNN
+F 0 "R1303" V 3407 4150 50  0000 C CNN
 F 1 "33R" V 3316 4150 50  0000 C CNN
 F 2 "Resistor_SMD:R_0805_2012Metric_Pad1.20x1.40mm_HandSolder" V 3130 4150 50  0001 C CNN
@@
 $EndComp
 $Comp
-L Device:R R1104
+L Device:R R1304
 U 1 1 614BBB41
 P 3200 4500
-F 0 "R1104" V 2993 4500 50  0000 C CNN
+F 0 "R1304" V 2993 4500 50  0000 C CNN
 F 1 "33R" V 3084 4500 50  0000 C CNN
 F 2 "Resistor_SMD:R_0805_2012Metric_Pad1.20x1.40mm_HandSolder" V 3130 4500 50  0001 C CNN
@@
 	8800 3250 9100 3250
 $Comp
-L Device:R R1102
+L Device:R R1302
 U 1 1 6163E3A9
 P 3200 3800
-F 0 "R1102" V 2993 3800 50  0000 C CNN
+F 0 "R1302" V 2993 3800 50  0000 C CNN
 F 1 "33R" V 3084 3800 50  0000 C CNN
 F 2 "Resistor_SMD:R_0805_2012Metric_Pad1.20x1.40mm_HandSolder" V 3130 3800 50  0001 C CNN
@@
 $EndComp
 $Comp
-L Device:R R1101
+L Device:R R1301
 U 1 1 6163F388
 P 3200 3450
-F 0 "R1101" V 2993 3450 50  0000 C CNN
+F 0 "R1301" V 2993 3450 50  0000 C CNN
 F 1 "33R" V 3084 3450 50  0000 C CNN
 F 2 "Resistor_SMD:R_0805_2012Metric_Pad1.20x1.40mm_HandSolder" V 3130 3450 50  0001 C CNN
@@
 Connection ~ 5350 2450
 $Comp
-L Device:R R1106
+L Device:R R1306
 U 1 1 6165B6E9
 P 4350 4700
-F 0 "R1106" H 4420 4746 50  0000 L CNN
+F 0 "R1306" H 4420 4746 50  0000 L CNN
 F 1 "10K" H 4420 4655 50  0000 L CNN
 F 2 "Resistor_SMD:R_0805_2012Metric_Pad1.20x1.40mm_HandSolder" V 4280 4700 50  0001 C CNN
@@
 $EndComp
 $Comp
-L Device:R R1105
+L Device:R R1305
 U 1 1 6165BF36
 P 3950 4700
-F 0 "R1105" H 4020 4746 50  0000 L CNN
+F 0 "R1305" H 4020 4746 50  0000 L CNN
 F 1 "10K" H 4020 4655 50  0000 L CNN
 F 2 "Resistor_SMD:R_0805_2012Metric_Pad1.20x1.40mm_HandSolder" V 3880 4700 50  0001 C CNN
