File: hw/led_holder/led_holder.kicad_pcb (KiCad board)
At the start: 2 copper layers, 5.8 x 11.6 mm, 7 parts, among them J1 Conn_01x01, J2 Conn_01x01, J3 Conn_01x01, J4 Conn_01x01

Commit message: [hw] Update led_holder to KiCad 6
Other:
- net class Default removed
