File: hw/simple_control/spi_sd_card.kicad_sch (KiCad schematic)
At the start: 7 parts, among them J6 Micro_SD_Card

Commit message: [hw] Add CPU modules
Connections:
- net +3V3 renamed +3.3V
Other:
- company: (none) -> Stefan Misik
- title: (none) -> WS2812 Simple Controller
Changed lines of the file:
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@@
 (kicad_sch (version 20230121) (generator eeschema)
   (paper "A4")
+  (title_block
+    (title "WS2812 Simple Controller")
+    (date "2023-03-09")
+    (company "Stefan Misik")
+    (comment 1 "SPI SD Card")
+  )
   (junction (at 111.76 64.77) (diameter 0) (color 0 0 0 0)
   )
@@
     )
   )
-  (symbol (lib_name "GND_2") (lib_id "power:GND") (at 111.76 115.57 0) (unit 1)
+  (symbol (lib_id "power:GND") (at 111.76 115.57 0) (unit 1)
     (in_bom yes) (on_board yes) (dnp no)
     (property "Reference" "#PWR033" (at 111.76 121.92 0)
@@
     )
   )
-  (symbol (lib_name "GND_1") (lib_id "power:GND") (at 179.07 114.3 0) (unit 1)
+  (symbol (lib_id "power:GND") (at 179.07 114.3 0) (unit 1)
     (in_bom yes) (on_board yes) (dnp no)
     (property "Reference" "#PWR035" (at 179.07 120.65 0)
